Commit message: delete arm and kinect

File: mm_description/urdf/mm.urdf.xacro (robot description, xacro)
@@ -3,33 +3,11 @@
   <!-- argument -->
   <xacro:arg name="robot_namespace" default="/"/>
-  <xacro:arg name="kinect1_enabled" default="true"/>
-  <xacro:arg name="kinect2_enabled" default="true"/>
-  <xacro:arg name="ur_enabled" default="true"/>
-  <xacro:arg name="gripper_enabled" default="true"/>
+  <xacro:arg name="kinect1_enabled" default="false"/>
+  <xacro:arg name="kinect2_enabled" default="false"/>
+  <xacro:arg name="ur_enabled" default="false"/>
+  <xacro:arg name="gripper_enabled" default="false"/>
   <!-- inspector_bot -->
   <xacro:include filename="$(find mm_description)/urdf/components/inspector_bot.urdf.xacro" />
   <xacro:include filename="$(find mm_description)/urdf/accessories/kinect_tilted_camera.urdf.xacro"/>
-  <xacro:include filename="$(find ur_description)/urdf/ur5.urdf.xacro" />
-  <xacro:include filename="$(find robotiq_2f_85_gripper_visualization)/urdf/robotiq_arg2f_85_model_macro.xacro" />
-  <!-- ur5 robot -->
-  <xacro:if value="$(arg ur_enabled)">
-    <xacro:property name="ur5_z_location" value="${base_center_height + base_z_size/2}" />
-    <xacro:property name="ur5_x_location" value="0.175" />
-    <joint name="ur_fixed_joint" type="fixed">
-      <parent link="bare_base_link" />
-      <child link="base_link" />
-      <origin xyz="${ur5_x_location} 0.0 ${ur5_z_location}" rpy="0.0 0.0 -${M_PI/2}" />
-    </joint>
-    <xacro:ur5_robot prefix="" joint_limited="false"/>
-    <!-- gripper -->
-    <xacro:if value="$(arg gripper_enabled)">
-      <joint name="ur_gripper_fixed_joint" type="fixed">
-        <parent link="tool0"/>
-        <child link="robotiq_arg2f_base_link"/>
-        <origin xyz="0 0 0" rpy="0 0 0"/>
-      </joint>
-      <xacro:robotiq_arg2f_85 prefix=""/>
-    </xacro:if>
-  </xacro:if>
   <!-- kinect -->
   <xacro:if value="$(arg kinect1_enabled)">

Commit message: mm default false

File: mm_description/urdf/mm.urdf.xacro (robot description, xacro)
@@ -3,6 +3,6 @@
   <!-- argument -->
   <xacro:arg name="robot_namespace" default="/"/>
-  <xacro:arg name="kinect1_enabled" default="true"/>
-  <xacro:arg name="kinect2_enabled" default="true"/>
+  <xacro:arg name="kinect1_enabled" default="false"/>
+  <xacro:arg name="kinect2_enabled" default="false"/>
   <xacro:arg name="ur_enabled" default="false"/>
   <xacro:arg name="gripper_enabled" default="false"/>
@@ -10,4 +10,26 @@
   <xacro:include filename="$(find mm_description)/urdf/components/inspector_bot.urdf.xacro" />
   <xacro:include filename="$(find mm_description)/urdf/accessories/kinect_tilted_camera.urdf.xacro"/>
+  <xacro:include filename="$(find ur_description)/urdf/ur5.urdf.xacro" />
+  <xacro:include filename="$(find robotiq_2f_85_gripper_visualization)/urdf/robotiq_arg2f_85_model_macro.xacro" />
+  <!-- ur5 robot -->
+  <xacro:if value="$(arg ur_enabled)">
+    <xacro:property name="ur5_z_location" value="${base_center_height + base_z_size/2}" />
+    <xacro:property name="ur5_x_location" value="0.175" />
+    <joint name="ur_fixed_joint" type="fixed">
+      <parent link="bare_base_link" />
+      <child link="base_link" />
+      <origin xyz="${ur5_x_location} 0.0 ${ur5_z_location}" rpy="0.0 0.0 -${M_PI/2}" />
+    </joint>
+    <xacro:ur5_robot prefix="" joint_limited="false"/>
+    <!-- gripper -->
+    <xacro:if value="$(arg gripper_enabled)">
+      <joint name="ur_gripper_fixed_joint" type="fixed">
+        <parent link="tool0"/>
+        <child link="robotiq_arg2f_base_link"/>
+        <origin xyz="0 0 0" rpy="0 0 0"/>
+      </joint>
+      <xacro:robotiq_arg2f_85 prefix=""/>
+    </xacro:if>
+  </xacro:if>
   <!-- kinect -->
   <xacro:if value="$(arg kinect1_enabled)">

Commit message: change ur5 ee

File: mm_description/urdf/mm.urdf.xacro (robot description, xacro)
@@ -29,4 +29,10 @@
         <origin xyz="0 0 0" rpy="0 0 0"/>
       </joint>
+      <joint name="ur_ee_fixed_joint" type="fixed">
+        <parent link="tool0"/>
+        <child link="robotiq_ee"/>
+        <origin xyz="0 0 0.15" rpy="0 0 0"/>
+      </joint>
+      <link name="robotiq_ee"/>
       <xacro:robotiq_arg2f_85 prefix=""/>
     </xacro:if>

Commit message: demo 01/10

File: mm_description/urdf/mm.urdf.xacro (robot description, xacro)
@@ -76,3 +76,22 @@
     </xacro:sensor_d435>
   </xacro:if>
+<!--
+  <joint name="test_fixed_joint" type="fixed">
+    <parent link="bare_base_link"/>
+    <child link="test_link"/>
+    <origin xyz = "0.0 -0.6 0.8" rpy="0 0 0"/>
+  </joint>
+  <link name="test_link">
+    <visual>
+      <geometry>
+        <cylinder length="0.3" radius="0.1"/>
+      </geometry>
+    </visual>
+    <collision>
+      <geometry>
+        <cylinder length="0.3" radius="0.1"/>
+      </geometry>
+    </collision>
+  </link>
+ -->
 </robot>

Commit message: v1.0.1 solved eef orientation problem - changed robotiq_ee tf in mm.urdf - changed gripper mesh(robotiq_2f85_opened_combined_axis_mated.STL) - added visualizing interactive marker gripper mesh

File: mm_description/urdf/mm.urdf.xacro (robot description, xacro)
@@ -31,8 +31,9 @@
         <origin xyz="0 0 0" rpy="0 0 0"/>
       </joint>
+      <!-- actual end-effector -->
       <joint name="ur_ee_fixed_joint" type="fixed">
         <parent link="tool0"/>
         <child link="robotiq_ee"/>
-        <origin xyz="0 0 0.125" rpy="0 0 0"/>
+        <origin xyz="0 0 0.13" rpy="0 -${M_PI/2} 0"/>
       </joint>
       <link name="robotiq_ee"/>

Commit message: v2.2 select IK solution(checkbox)

File: mm_description/urdf/mm.urdf.xacro (robot description, xacro)
@@ -23,4 +23,10 @@
       <origin xyz="${ur5_x_location} 0.0 ${ur5_z_location}" rpy="0.0 0.0 -${M_PI/2}" />
     </joint>
+    <joint name="ur_real_ee_fixed_joint" type="fixed">
+      <parent link="ee_link" />
+      <child link="real_ee_link" />
+      <origin xyz="0.0 0.0 0.0" rpy="-${M_PI/2} 0.0 -${M_PI/2}" />
+    </joint>
+    <link name="real_ee_link"/>
     <xacro:ur5_robot prefix="" joint_limited="false"/>
     <!-- gripper -->

Commit message: move xyz wrt eef

File: mm_description/urdf/mm.urdf.xacro (robot description, xacro)
@@ -83,22 +83,3 @@
     </xacro:sensor_d435>
   </xacro:if>
-<!--
-  <joint name="test_fixed_joint" type="fixed">
-    <parent link="bare_base_link"/>
-    <child link="test_link"/>
-    <origin xyz = "0.0 -0.6 0.8" rpy="0 0 0"/>
-  </joint>
-  <link name="test_link">
-    <visual>
-      <geometry>
-        <cylinder length="0.3" radius="0.1"/>
-      </geometry>
-    </visual>
-    <collision>
-      <geometry>
-        <cylinder length="0.3" radius="0.1"/>
-      </geometry>
-    </collision>
-  </link>
- -->
 </robot>
