Commit message: change imu axis

File: mm_description/urdf/components/inspector_bot.urdf.xacro (robot description, xacro)
@@ -86,5 +86,5 @@
   <link name="base_imu_link"/>
   <joint name="imu_joint" type="fixed">
-    <origin xyz="0 0 0" rpy="0 0 0" />
+    <origin xyz="0 0 0" rpy="0 0 ${3*M_PI/2}" />
     <parent link="bare_base_link" />
     <child link="base_imu_link" />

Commit message: tmp

File: mm_description/urdf/components/inspector_bot.urdf.xacro (robot description, xacro)
@@ -86,5 +86,5 @@
   <link name="base_imu_link"/>
   <joint name="imu_joint" type="fixed">
-    <origin xyz="0 0 0" rpy="0 0 ${3*M_PI/2}" />
+    <origin xyz="0 0 0" rpy="${M_PI} 0 0" />
     <parent link="bare_base_link" />
     <child link="base_imu_link" />

Commit message: add demo

File: mm_description/urdf/components/inspector_bot.urdf.xacro (robot description, xacro)
@@ -40,6 +40,6 @@
       </collision>
     </link>
-    <!-- <joint name="${wheel_prefix}_wheel" type="fixed"> -->
-    <joint name="${wheel_prefix}_wheel" type="continuous">
+    <joint name="${wheel_prefix}_wheel" type="fixed">
+    <!-- <joint name="${wheel_prefix}_wheel" type="continuous"> -->
       <xacro:insert_block name="joint_pose"/>
       <parent link="bare_base_link"/>
@@ -90,4 +90,11 @@
     <child link="base_imu_link" />
   </joint>
+  <!-- laser link -->
+  <link name="base_laser_link"/>
+  <joint name="laser_joint" type="fixed">
+    <origin xyz="${base_x_size/2+0.1} 0 ${wheel_radius*2}" rpy="0 0 0" />
+    <parent link="bare_base_link" />
+    <child link="base_laser_link" />
+  </joint>
   <!-- inspector_bot wheels -->
   <xacro:inspector_bot_wheel wheel_prefix="front_left">

File: mm_description/urdf/mm.urdf.xacro (robot description, xacro)
@@ -4,5 +4,6 @@
   <xacro:arg name="robot_namespace" default="/"/>
   <xacro:arg name="kinect1_enabled" default="true"/>
-  <xacro:arg name="kinect2_enabled" default="true"/>
+  <xacro:arg name="kinect2_enabled" default="false"/>
+  <xacro:arg name="realsense_enabled" default="true"/>
   <xacro:arg name="ur_enabled" default="true"/>
   <xacro:arg name="gripper_enabled" default="true"/>
@@ -12,4 +13,5 @@
   <xacro:include filename="$(find ur_description)/urdf/ur5.urdf.xacro" />
   <xacro:include filename="$(find robotiq_2f_85_gripper_visualization)/urdf/robotiq_arg2f_85_model_macro.xacro" />
+  <xacro:include filename="$(find realsense2_description)/urdf/_d435.urdf.xacro" />
   <!-- ur5 robot -->
   <xacro:if value="$(arg ur_enabled)">
@@ -32,5 +34,5 @@
         <parent link="tool0"/>
         <child link="robotiq_ee"/>
-        <origin xyz="0 0 0.15" rpy="0 0 0"/>
+        <origin xyz="0 0 0.125" rpy="0 0 0"/>
       </joint>
       <link name="robotiq_ee"/>
@@ -56,3 +58,21 @@
       base_xyz="$(arg kinect2_base_xyz)" base_rpy="$(arg kinect2_base_rpy)" tilt_angle="$(arg kinect2_tilt_angle)"/>
   </xacro:if>
+  <xacro:if value="$(arg realsense_enabled)">
+    <xacro:property name="realsense_height" value="${0.415+0.077}"/>
+    <link name="realsense_mount_link" />
+    <joint name="base_realsense_fixed_joint" type="fixed">
+      <parent link="bare_base_link"/>
+      <child link="realsense_mount_link"/>
+      <origin xyz="${-base_x_size/2 - profile_size/2} ${-base_y_size/2 + profile_size*1.5} ${base_center_height + base_z_size/2 + realsense_height}" rpy="0 0 ${-M_PI/4}"/>
+    </joint>
+    <link name="realsense_base_link" />
+    <joint name="realsense_mount_fixed_joint" type="fixed">
+      <parent link="realsense_mount_link"/>
+      <child link="realsense_base_link"/>
+      <origin xyz="0.035 0 0.025" rpy="0 ${M_PI/6} 0"/>
+    </joint>
+    <xacro:sensor_d435 parent="realsense_base_link">
+      <origin xyz="0.010 0 -0.0125" rpy="0 0 0"/>
+    </xacro:sensor_d435>
+  </xacro:if>
 </robot>

Commit message: v4.0 (demo on 0207)

File: mm_description/urdf/components/inspector_bot.urdf.xacro (robot description, xacro)
@@ -1,4 +1,6 @@
 <?xml version="1.0"?>
 <robot name="inspector_bot" xmlns:xacro="http://ros.org/wiki/xacro">
+  <!-- Materials -->
+  <xacro:include filename="$(find mm_description)/urdf/common_properties.xacro" />
   <!-- Base Size -->
   <xacro:property name="base_x_size" value="0.76" />
@@ -7,4 +9,5 @@
   <!-- Profile Size -->
   <xacro:property name="profile_size" value="0.04" />
+  <xacro:property name="profile_height1" value="${0.415+0.077}"/> <!-- camera -->
   <!-- Origin -->
   <xacro:property name="origin_x" value="0.025" />
@@ -61,5 +64,5 @@
         <box size = "${base_x_size}  ${base_y_size}  ${base_z_size}"/>
       </geometry>
-      <material name="white"/>
+      <material name="black"/>
     </visual>
     <collision>
@@ -110,3 +113,23 @@
     <origin xyz="${-wheelbase/2} ${-track/2} ${wheel_vertical_offset}" rpy="0 0 0" />
   </xacro:inspector_bot_wheel>
+  <!-- profile for side facing camera -->
+  <joint name="camera_profile_fixed_joint" type="fixed">
+    <parent link="bare_base_link"/>
+    <child link="camera_profile"/>
+    <origin xyz="${-base_x_size/2 - profile_size/2} ${-base_y_size/2 + profile_size*1.5} ${base_center_height + base_z_size/2 + profile_height1/2}" rpy="0 0 0"/>
+  </joint>
+  <link name="camera_profile">
+    <visual>
+      <geometry>
+        <box size="${profile_size} ${profile_size} ${profile_height1}"/>
+      </geometry>
+      <material name="black"/>
+    </visual>
+    <collision>
+      <geometry>
+        <box size="${profile_size} ${profile_size} ${profile_height1}"/>
+      </geometry>
+      <material name="black"/>
+    </collision>
+  </link>
 </robot>

File: mm_description/urdf/mm.urdf.xacro (robot description, xacro)
@@ -1,12 +1,13 @@
 <?xml version="1.0"?>
 <robot name="mobile_manipulator" xmlns:xacro="http://ros.org/wiki/xacro">
-  <!-- argument -->
+  <!-- arguments -->
   <xacro:arg name="robot_namespace" default="/"/>
   <xacro:arg name="kinect1_enabled" default="true"/>
   <xacro:arg name="kinect2_enabled" default="false"/>
-  <xacro:arg name="realsense_enabled" default="true"/>
+  <xacro:arg name="realsense1_enabled" default="true"/>
+  <xacro:arg name="realsense2_enabled" default="true"/>
   <xacro:arg name="ur_enabled" default="true"/>
   <xacro:arg name="gripper_enabled" default="true"/>
-  <!-- inspector_bot -->
+  <!-- components -->
   <xacro:include filename="$(find mm_description)/urdf/components/inspector_bot.urdf.xacro" />
   <xacro:include filename="$(find mm_description)/urdf/accessories/kinect_tilted_camera.urdf.xacro"/>
@@ -14,5 +15,8 @@
   <xacro:include filename="$(find robotiq_2f_85_gripper_visualization)/urdf/robotiq_arg2f_85_model_macro.xacro" />
   <xacro:include filename="$(find realsense2_description)/urdf/_d415.urdf.xacro" />
-  <!-- ur5 robot -->
+  <xacro:include filename="$(find realsense2_description)/urdf/_d435.urdf.xacro" />
+  <!-- ********************* -->
+  <!--          ur5          -->
+  <!-- ********************* -->
   <xacro:if value="$(arg ur_enabled)">
     <xacro:property name="ur5_z_location" value="${base_center_height + base_z_size/2}" />
@@ -47,5 +51,7 @@
     </xacro:if>
   </xacro:if>
-  <!-- kinect -->
+  <!-- ********************* -->
+  <!--         kinect        -->
+  <!-- ********************* -->
   <xacro:if value="$(arg kinect1_enabled)">
     <xacro:arg name="kinect1_base_xyz" default="${base_x_size/2 + 0.041} 0 ${base_center_height + base_z_size/2 - 0.071}"/>
@@ -65,12 +71,32 @@
       base_xyz="$(arg kinect2_base_xyz)" base_rpy="$(arg kinect2_base_rpy)" tilt_angle="$(arg kinect2_tilt_angle)"/>
   </xacro:if>
-  <xacro:if value="$(arg realsense_enabled)">
-    <link name="realsense_base_link" />
-    <joint name="realsense_mount_fixed_joint" type="fixed">
+  <!-- ********************* -->
+  <!--       realsense       -->
+  <!-- ********************* -->
+  <xacro:if value="$(arg realsense1_enabled)">
+    <link name="realsense1_mount_link" />
+    <joint name="realsense1_profile_fixed_joint" type="fixed">
+      <parent link="camera_profile"/>
+      <child link="realsense1_mount_link"/>
+      <origin xyz="0 0 ${profile_height1/2}" rpy="0 0 ${-M_PI/4}"/>
+    </joint>
+    <link name="realsense1_base_link" />
+    <joint name="realsense1_mount_fixed_joint" type="fixed">
+      <parent link="realsense1_mount_link"/>
+      <child link="realsense1_base_link"/>
+      <origin xyz="0.035 0 0.025" rpy="0 ${M_PI/6} 0"/>
+    </joint>
+    <xacro:sensor_d435 parent="realsense1_base_link" name="realsense1">
+      <origin xyz="0.010 0 -0.0125" rpy="0 0 0"/>
+    </xacro:sensor_d435>
+  </xacro:if>
+  <xacro:if value="$(arg realsense2_enabled)">
+    <link name="realsense2_base_link" />
+    <joint name="realsense2_mount_fixed_joint" type="fixed">
       <parent link="ee_link"/>
-      <child link="realsense_base_link"/>
-      <origin xyz="-0.02 0.077 0.0" rpy="${-M_PI/2} 0 0"/>
+      <child link="realsense2_base_link"/>
+      <origin xyz="-0.02 0.065 0.0" rpy="${-M_PI/2} 0 0"/>
     </joint>
-    <xacro:sensor_d415 parent="realsense_base_link">
+    <xacro:sensor_d415 parent="realsense2_base_link" name="realsense2">
       <origin xyz="0 0 0" rpy="0 0 0"/>
     </xacro:sensor_d415>

Commit message: v5.1 - test 03/04

File: mm_description/urdf/components/inspector_bot.urdf.xacro (robot description, xacro)
@@ -21,4 +21,8 @@
   <xacro:property name="wheel_radius" value="0.2" />
   <xacro:property name="base_center_height" value="${wheel_vertical_offset + wheel_radius}" />
+  <!-- Battery Size -->
+  <xacro:property name="battery_x_size" value="${0.18+0.02}"/>
+  <xacro:property name="battery_y_size" value="${0.36+0.02}"/>
+  <xacro:property name="battery_z_size" value="${0.28+0.02}"/>
   <xacro:property name="M_PI" value="3.14159"/>
   <!-- Inspector_bot wheel macro -->
@@ -54,5 +58,6 @@
   <link name="base_footprint"/>
   <joint name="base_joint" type="fixed">
-    <origin xyz="-${base_x_size/2 + origin_x} ${base_y_size/2 - origin_y} 0" rpy="0 0 0" />
+    <!-- <origin xyz="-${base_x_size/2 + origin_x} ${base_y_size/2 - origin_y} 0" rpy="0 0 0" /> -->
+    <origin xyz="0 0 0" rpy="0 0 0" />
     <parent link="base_footprint" />
     <child link="bare_base_link" />
@@ -114,5 +119,5 @@
   </xacro:inspector_bot_wheel>
   <!-- profile for side facing camera -->
-  <joint name="camera_profile_fixed_joint" type="fixed">
+  <!-- <joint name="camera_profile_fixed_joint" type="fixed">
     <parent link="bare_base_link"/>
     <child link="camera_profile"/>
@@ -132,4 +137,24 @@
       <material name="black"/>
     </collision>
+  </link> -->
+  <!-- battery -->
+  <joint name="camera_profile_fixed_joint" type="fixed">
+    <parent link="bare_base_link"/>
+    <child link="battery_link"/>
+    <origin xyz="${-base_x_size/2 + profile_size + battery_x_size/2} 0 ${base_center_height + base_z_size/2 + battery_z_size/2}" rpy="0 0 0"/>
+  </joint>
+  <link name="battery_link">
+    <visual>
+      <geometry>
+        <box size="${battery_x_size} ${battery_y_size} ${battery_z_size}"/>
+      </geometry>
+      <material name="black"/>
+    </visual>
+    <collision>
+      <geometry>
+        <box size="${battery_x_size} ${battery_y_size} ${battery_z_size}"/>
+      </geometry>
+      <material name="black"/>
+    </collision>
   </link>
 </robot>

File: mm_description/urdf/mm.urdf.xacro (robot description, xacro)
@@ -5,5 +5,5 @@
   <xacro:arg name="kinect1_enabled" default="true"/>
   <xacro:arg name="kinect2_enabled" default="false"/>
-  <xacro:arg name="realsense1_enabled" default="true"/>
+  <xacro:arg name="realsense1_enabled" default="false"/>
   <xacro:arg name="realsense2_enabled" default="true"/>
   <xacro:arg name="ur_enabled" default="true"/>

Commit message: gui changes

File: mm_description/urdf/components/inspector_bot.urdf.xacro (robot description, xacro)
@@ -95,4 +95,5 @@
   <joint name="imu_joint" type="fixed">
     <origin xyz="0 0 0" rpy="${M_PI} 0 0" />
+    <!-- <origin xyz="0 0 0" rpy="0 0 0" /> -->
     <parent link="bare_base_link" />
     <child link="base_imu_link" />
